File: CS5464_Breakout.kicad_pcb (KiCad board)
At the start: 2 copper layers, 35.6 x 27.9 mm, 37 parts, among them J1 Conn_01x10, U1 CS5464-ISZ, Y1 4.096MHz

Commit message: Add silk screen and shorted test pad name, bump version
Parts:
- moved LOGO1 0.76 mm to (133.9, 93.3)
- renumbered CPUCLK1 to CCLK1
Other:
- board text added: "3V3"
- board text added: "GND"
- board text added: "IN"
- board text added: "IP"
- board text added: "MISO"
- board text added: "MOSI"
- board text added: "SCLK"
- board text added: "VN"
- board text added: "VP"
- board text added: "by Tisham Dhar http://whatnick.com v0.2 19/01/2020"
- board text added: "~CS"
- board text removed: "by Tisham Dhar http://whatnick.com v0.1 06/02/2019"
